File: rw-piggyback.kicad_pcb (KiCad board)
At the start: 2 copper layers, 125.7 x 77.5 mm, 8 parts, among them J1 Logic Board, J2 RAM Card, J3 Piggyback A, J4 Piggyback B, J5 Power, J6 USB A

Commit message: Repoint
Parts:
- G1: footprint pub:piggyback-logo-2 -> rharke:piggyback-logo-2
- J1: footprint pub:AppleIIeAux -> rharke:AppleIIeAux
- J2: footprint pub:CardEdge_EDAC_3x5-060_2x30_P2.54mm_CCW_No47 -> rharke:CardEdge_EDAC_3x5-060_2x30_P2.54mm_CCW_No47
- J6: footprint pub:USB_A_Stewart_SS-52100-001_Horizontal -> rharke:USB_A_Stewart_SS-52100-001_Horizontal
Changed lines of the file:
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@@
     (add_net GND)
   )
-  (module pub:piggyback-logo-2 (layer F.Cu)
+  (module rharke:piggyback-logo-2 (layer F.Cu)
     (at 109.22 132.715)
     (fp_text reference G1 (at 0 0) (layer F.SilkS) hide
@@
       (xy -2.356701 -8.330373)) (layer F.SilkS) (width 0.01))
   )
-  (module pub:USB_A_Stewart_SS-52100-001_Horizontal (layer F.Cu)
+  (module rharke:USB_A_Stewart_SS-52100-001_Horizontal (layer F.Cu)
     (at 194.945 81.28 90)
     (descr "USB A connector https://belfuse.com/resources/drawings/stewartconnector/dr-stw-ss-52100-001.pdf")
@@
     )
   )
-  (module pub:CardEdge_EDAC_3x5-060_2x30_P2.54mm_CCW_No47 (layer F.Cu)
+  (module rharke:CardEdge_EDAC_3x5-060_2x30_P2.54mm_CCW_No47 (layer F.Cu)
     (at 116.205 127 90)
     (descr "Through hole straight pin header, 2x25, 2.54mm pitch, double rows")
@@
     )
   )
-  (module pub:AppleIIeAux (layer F.Cu)
+  (module rharke:AppleIIeAux (layer F.Cu)
     (at 108.585 133.985)
     (fp_text reference J1 (at 36.83 -5.08) (layer F.SilkS) hide
